Commit message: broken gazebo

File: ros/robocock/description/robot_core.xacro (robot description, xacro)
@@ -168,8 +168,46 @@
     </gazebo>
     <!-- Transmissions -->
-    <!-- Make Gazebo publish joint states -->
+    <transmission name="tran1">
+        <type>transmission_interface/SimpleTransmission</type>
+        <joint name="wheel_1_joint">
+            <hardwareInterface>hardware_interface/VelocityJointInterface</hardwareInterface>
+        </joint>
+        <actuator name="motor_1">
+            <hardwareInterface>VelocityJointInterface</hardwareInterface>
+            <mechanicalReduction>1</mechanicalReduction>
+        </actuator>
+    </transmission>
+    <transmission name="tran2">
+        <type>transmission_interface/SimpleTransmission</type>
+        <joint name="wheel_2_joint">
+            <hardwareInterface>hardware_interface/VelocityJointInterface</hardwareInterface>
+        </joint>
+        <actuator name="motor_2">
+            <hardwareInterface>VelocityJointInterface</hardwareInterface>
+            <mechanicalReduction>1</mechanicalReduction>
+        </actuator>
+    </transmission>
+    <transmission name="tran3">
+        <type>transmission_interface/SimpleTransmission</type>
+        <joint name="wheel_3_joint">
+            <hardwareInterface>hardware_interface/VelocityJointInterface</hardwareInterface>
+        </joint>
+        <actuator name="motor_3">
+            <hardwareInterface>VelocityJointInterface</hardwareInterface>
+            <mechanicalReduction>1</mechanicalReduction>
+        </actuator>
+    </transmission>
+    <transmission name="tran4">
+        <type>transmission_interface/SimpleTransmission</type>
+        <joint name="wheel_4_joint">
+            <hardwareInterface>hardware_interface/VelocityJointInterface</hardwareInterface>
+        </joint>
+        <actuator name="motor_4">
+            <hardwareInterface>VelocityJointInterface</hardwareInterface>
+            <mechanicalReduction>1</mechanicalReduction>
+        </actuator>
+    </transmission>
     <gazebo>
         <plugin name="gazebo_ros_control" filename="libgazebo_ros_control.so">
-            <robotNamespace>/</robotNamespace>
         </plugin>
     </gazebo>

Commit message: added laser

File: ros/robocock/description/robot_core.xacro (robot description, xacro)
@@ -11,5 +11,5 @@
         <child link="chassis"/>
         <origin xyz="0 0 0"/>
-    </joint>
+    </joint> launch-prefix="bash -c 'sleep 5; $0 $@'"
     <!-- chassis description goes here. It describes the chassis of robocock which is a 54cm x 54cm x 150cm box -->
     <link name="chassis">
@@ -35,4 +35,18 @@
         </xacro:inertial_box>
     </link>
+    <joint name="laser_joint" type="fixed">
+        <parent link="chassis"/>
+        <child link="laser"/>
+        <origin xyz="0.25 0 0.5" rpy="0 0 0"/>
+    </joint>
+    <link name="laser">
+        <visual>
+            <origin xyz="0 0 0" rpy="0 0 0"/>
+            <geometry>
+                <cylinder length="0.05" radius="0.05"/>
+            </geometry>
+            <material name="black"/>
+        </visual>
+    </link>
     <!-- gazebo specific description -->
     <gazebo reference="chassis">

Commit message: slam stuff

File: ros/robocock/description/robot_core.xacro (robot description, xacro)
@@ -38,5 +38,5 @@
         <parent link="chassis"/>
         <child link="laser"/>
-        <origin xyz="0.25 0 0.5" rpy="0 0 0"/>
+        <origin xyz="-0.25 0 0.5" rpy="0 0 0"/>
     </joint>
     <link name="laser">
