File: circuits/motor_controller.kicad_sch (KiCad schematic)
At the start: 0 parts

Commit message: motor shield circuit
BTN7030-1EPA
Parts:
- added A1: A000067, ARDUINO_A000067, symbol A000067:A000067
- added J3: Conn_01x03_Pin, symbol Connector:Conn_01x03_Pin
- added R6: 1k6, symbol Device:R_Small
- added R7: 3k3, symbol Device:R_Small
Connections:
- new net: A1.14, R6.1
- new net +5V: A1.5V_1 (+5V_1)
- new net 1_HALL_A: A1.18
- new net 1_HALL_B: A1.30
- new net 1_IS: A1.AD0
- new net 1_LPWM: A1.2
- new net 1_RPWM: A1.7
- new net 2_HALL_A: A1.19
- new net 2_HALL_B: A1.31
- new net 2_LPWM: A1.3
- new net 2_RPWM: A1.8
- new net 3_HALL_A: A1.20
- new net 3_HALL_B: A1.32
- new net 3_LPWM: A1.5
- new net 3_RPWM: A1.11
- new net 4_HALL_A: A1.21
- new net 4_HALL_B: A1.33
- new net 4_LPWM: A1.6
- new net 4_RPWM: A1.12
- new net GND: A1.GND1, J3.3 (Pin_3), R7.2
- new net PI_RX: J3.2 (Pin_2), R6.2, R7.1
- new net PI_TX: A1.15, J3.1 (Pin_1)
- no-connect marks 0 -> 1
Other:
- note added: "Raspberry Pi UART"

Commit message: controller pcb rev 1
Parts:
- removed J3: Conn_01x03_Pin, symbol Connector:Conn_01x03_Pin
- added J?: Conn_01x02_Pin, Connector_PinHeader_2.54mm:PinHeader_1x02_P2.54mm_Vertical, symbol Connector:Conn_01x02_Pin
- A1: footprint ARDUINO_A000067 -> A000067:ARDUINO_A000067
- R5: renamed from R6; footprint (none) -> Resistor_SMD:R_0805_2012Metric_Pad1.20x1.40mm_HandSolder
- R6: renamed from R7; footprint (none) -> Resistor_SMD:R_1206_3216Metric_Pad1.30x1.75mm_HandSolder
Connections:
- net PI_RX: now also J?.2 (Pin_2)
- net PI_TX: now also J?.1 (Pin_1)
- net 2_IS: now reaches A1.AD1
- net 3_IS: now reaches A1.AD2
- net 4_IS: now reaches A1.AD3
- no-connect marks 1 -> 62
Changed lines of the file:
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@@
   (junction (at 152.4 111.76) (diameter 0) (color 0 0 0 0)
   )
+  (no_connect (at 137.16 147.32))
+  (no_connect (at 96.52 86.36))
+  (no_connect (at 96.52 76.2))
+  (no_connect (at 96.52 127))
+  (no_connect (at 137.16 96.52))
+  (no_connect (at 137.16 119.38))
+  (no_connect (at 137.16 132.08))
+  (no_connect (at 96.52 129.54))
+  (no_connect (at 96.52 116.84))
+  (no_connect (at 137.16 116.84))
+  (no_connect (at 137.16 53.34))
+  (no_connect (at 96.52 43.18))
+  (no_connect (at 96.52 55.88))
+  (no_connect (at 96.52 114.3))
+  (no_connect (at 96.52 99.06))
+  (no_connect (at 96.52 73.66))
+  (no_connect (at 96.52 142.24))
+  (no_connect (at 96.52 45.72))
+  (no_connect (at 96.52 58.42))
+  (no_connect (at 96.52 101.6))
+  (no_connect (at 96.52 93.98))
+  (no_connect (at 137.16 45.72))
+  (no_connect (at 96.52 111.76))
+  (no_connect (at 96.52 139.7))
+  (no_connect (at 137.16 99.06))
+  (no_connect (at 96.52 147.32))
+  (no_connect (at 137.16 81.28))
+  (no_connect (at 96.52 81.28))
+  (no_connect (at 137.16 127))
+  (no_connect (at 137.16 71.12))
+  (no_connect (at 137.16 137.16))
+  (no_connect (at 96.52 88.9))
+  (no_connect (at 137.16 144.78))
   (no_connect (at 96.52 40.64))
+  (no_connect (at 137.16 78.74))
+  (no_connect (at 137.16 142.24))
+  (no_connect (at 137.16 152.4))
+  (no_connect (at 96.52 132.08))
+  (no_connect (at 137.16 35.56))
+  (no_connect (at 137.16 114.3))
+  (no_connect (at 96.52 149.86))
+  (no_connect (at 96.52 119.38))
+  (no_connect (at 96.52 134.62))
+  (no_connect (at 96.52 96.52))
+  (no_connect (at 137.16 111.76))
+  (no_connect (at 96.52 144.78))
+  (no_connect (at 137.16 109.22))
+  (no_connect (at 96.52 104.14))
+  (no_connect (at 96.52 48.26))
+  (no_connect (at 137.16 40.64))
+  (no_connect (at 96.52 109.22))
+  (no_connect (at 137.16 139.7))
+  (no_connect (at 137.16 129.54))
+  (no_connect (at 137.16 55.88))
+  (no_connect (at 96.52 152.4))
+  (no_connect (at 137.16 134.62))
+  (no_connect (at 96.52 78.74))
+  (no_connect (at 137.16 43.18))
+  (no_connect (at 96.52 91.44))
+  (no_connect (at 137.16 38.1))
+  (no_connect (at 96.52 137.16))
+  (no_connect (at 137.16 149.86))
   (wire (pts (xy 88.9 50.8) (xy 96.52 50.8))
     (stroke (width 0) (type default))
@@
   )
   (wire (pts (xy 152.4 111.76) (xy 154.94 111.76))
-    (stroke (width 0) (type default))
-  )
-  (wire (pts (xy 151.13 182.88) (xy 154.94 182.88))
     (stroke (width 0) (type default))
   )
@@
     )
   )
+  (global_label "2_IS" (shape input) (at 96.52 66.04 180) (fields_autoplaced)
+    (effects (font (size 1.27 1.27)) (justify right))
+    (property "Intersheetrefs" "${INTERSHEET_REFS}" (at 89.5434 66.04 0)
+      (effects (font (size 1.27 1.27)) (justify right) hide)
+    )
+  )
   (global_label "1_RPWM" (shape input) (at 137.16 63.5 0) (fields_autoplaced)
     (effects (font (size 1.27 1.27)) (justify left))
@@
     (property "Intersheetrefs" "${INTERSHEET_REFS}" (at 147.4438 73.66 0)
       (effects (font (size 1.27 1.27)) (justify left) hide)
+    )
+  )
+  (global_label "3_IS" (shape input) (at 96.52 68.58 180) (fields_autoplaced)
+    (effects (font (size 1.27 1.27)) (justify right))
+    (property "Intersheetrefs" "${INTERSHEET_REFS}" (at 89.5434 68.58 0)
+      (effects (font (size 1.27 1.27)) (justify right) hide)
     )
   )
@@
     )
   )
+  (global_label "4_IS" (shape input) (at 96.52 71.12 180) (fields_autoplaced)
+    (effects (font (size 1.27 1.27)) (justify right))
+    (property "Intersheetrefs" "${INTERSHEET_REFS}" (at 89.5434 71.12 0)
+      (effects (font (size 1.27 1.27)) (justify right) hide)
+    )
+  )
   (global_label "3_HALL_B" (shape input) (at 137.16 124.46 0) (fields_autoplaced)
     (effects (font (size 1.27 1.27)) (justify left))
@@
       (effects (font (size 1.27 1.27)))
     )
-    (property "Footprint" "ARDUINO_A000067" (at 116.84 93.98 0)
+    (property "Footprint" "A000067:ARDUINO_A000067" (at 116.84 93.98 0)
       (effects (font (size 1.27 1.27)) (justify bottom) hide)
     )
@@
   (symbol (lib_id "power:GND") (at 88.9 53.34 0) (unit 1)
     (in_bom yes) (on_board yes) (dnp no) (fields_autoplaced)
-    (property "Reference" "#PWR013" (at 88.9 59.69 0)
+    (property "Reference" "#PWR012" (at 88.9 59.69 0)
       (effects (font (size 1.27 1.27)) hide)
     )
@@
       (project "rbc_circuits"
         (path "/1df96114-eb1a-4ddf-9ea3-acd2b4d12bf3/11663713-acec-45f1-8603-bba89fd94900"
-          (reference "#PWR013") (unit 1)
+          (reference "#PWR012") (unit 1)
+        )
+      )
+    )
+  )
+  (symbol (lib_id "Connector:Conn_01x02_Pin") (at 146.05 177.8 0) (unit 1)
+    (in_bom yes) (on_board yes) (dnp no)
+    (property "Reference" "J?" (at 147.32 175.26 0)
+      (effects (font (size 1.27 1.27)))
+    )
+    (property "Value" "Conn_01x02_Pin" (at 146.685 175.26 0)
+      (effects (font (size 1.27 1.27)) hide)
+    )
+    (property "Footprint" "Connector_PinHeader_2.54mm:PinHeader_1x02_P2.54mm_Vertical" (at 146.05 177.8 0)
+      (effects (font (size 1.27 1.27)) hide)
+    )
+    (property "Datasheet" "~" (at 146.05 177.8 0)
+      (effects (font (size 1.27 1.27)) hide)
+    )
+    (pin "1")
+    (pin "2")
+    (instances
+      (project "rbc_circuits"
+        (path "/1df96114-eb1a-4ddf-9ea3-acd2b4d12bf3/6683f276-27a3-494e-84c3-353277da8be6"
+          (reference "J?") (unit 1)
+        )
+        (path "/1df96114-eb1a-4ddf-9ea3-acd2b4d12bf3/11663713-acec-45f1-8603-bba89fd94900"
+          (reference "J3") (unit 1)
         )
       )
@@
   (symbol (lib_id "power:GND") (at 152.4 118.11 0) (unit 1)
     (in_bom yes) (on_board yes) (dnp no) (fields_autoplaced)
-    (property "Reference" "#PWR012" (at 152.4 124.46 0)
+    (property "Reference" "#PWR013" (at 152.4 124.46 0)
       (effects (font (size 1.27 1.27)) hide)
     )
@@
       (project "rbc_circuits"
         (path "/1df96114-eb1a-4ddf-9ea3-acd2b4d12bf3/11663713-acec-45f1-8603-bba89fd94900"
-          (reference "#PWR012") (unit 1)
-        )
-      )
-    )
-  )
-  (symbol (lib_id "Connector:Conn_01x03_Pin") (at 146.05 180.34 0) (unit 1)
-    (in_bom yes) (on_board yes) (dnp no) (fields_autoplaced)
-    (property "Reference" "J3" (at 146.685 176.53 0)
-      (effects (font (size 1.27 1.27)))
-    )
-    (property "Value" "Conn_01x03_Pin" (at 146.685 176.53 0)
-      (effects (font (size 1.27 1.27)) hide)
-    )
-    (property "Footprint" "" (at 146.05 180.34 0)
-      (effects (font (size 1.27 1.27)) hide)
-    )
-    (property "Datasheet" "~" (at 146.05 180.34 0)
-      (effects (font (size 1.27 1.27)) hide)
-    )
-    (pin "1")
-    (pin "2")
-    (pin "3")
-    (instances
-      (project "rbc_circuits"
-        (path "/1df96114-eb1a-4ddf-9ea3-acd2b4d12bf3/11663713-acec-45f1-8603-bba89fd94900"
-          (reference "J3") (unit 1)
+          (reference "#PWR013") (unit 1)
         )
       )
@@
   (symbol (lib_id "Device:R_Small") (at 152.4 107.95 0) (unit 1)
     (in_bom yes) (on_board yes) (dnp no)
-    (property "Reference" "R6" (at 147.32 106.68 0)
+    (property "Reference" "R5" (at 147.32 106.68 0)
       (effects (font (size 1.27 1.27)) (justify left))
     )
@@
       (effects (font (size 1.27 1.27)) (justify left))
     )
-    (property "Footprint" "" (at 152.4 107.95 0)
+    (property "Footprint" "Resistor_SMD:R_0805_2012Metric_Pad1.20x1.40mm_HandSolder" (at 152.4 107.95 0)
       (effects (font (size 1.27 1.27)) hide)
     )
@@
       (project "rbc_circuits"
         (path "/1df96114-eb1a-4ddf-9ea3-acd2b4d12bf3/11663713-acec-45f1-8603-bba89fd94900"
-          (reference "R6") (unit 1)
+          (reference "R5") (unit 1)
         )
       )
@@
     )
   )
-  (symbol (lib_id "power:GND") (at 154.94 182.88 0) (unit 1)
-    (in_bom yes) (on_board yes) (dnp no) (fields_autoplaced)
-    (property "Reference" "#PWR014" (at 154.94 189.23 0)
-      (effects (font (size 1.27 1.27)) hide)
-    )
-    (property "Value" "GND" (at 154.94 187.96 0)
-      (effects (font (size 1.27 1.27)))
-    )
-    (property "Footprint" "" (at 154.94 182.88 0)
-      (effects (font (size 1.27 1.27)) hide)
-    )
-    (property "Datasheet" "" (at 154.94 182.88 0)
-      (effects (font (size 1.27 1.27)) hide)
-    )
-    (pin "1")
-    (instances
-      (project "rbc_circuits"
-        (path "/1df96114-eb1a-4ddf-9ea3-acd2b4d12bf3/11663713-acec-45f1-8603-bba89fd94900"
-          (reference "#PWR014") (unit 1)
-        )
-      )
-    )
-  )
   (symbol (lib_id "Device:R_Small") (at 152.4 115.57 0) (unit 1)
     (in_bom yes) (on_board yes) (dnp no)
-    (property "Reference" "R7" (at 147.32 114.3 0)
+    (property "Reference" "R6" (at 147.32 114.3 0)
       (effects (font (size 1.27 1.27)) (justify left))
     )
@@
       (effects (font (size 1.27 1.27)) (justify left))
     )
-    (property "Footprint" "" (at 152.4 115.57 0)
+    (property "Footprint" "Resistor_SMD:R_1206_3216Metric_Pad1.30x1.75mm_HandSolder" (at 152.4 115.57 0)
       (effects (font (size 1.27 1.27)) hide)
     )
@@
       (project "rbc_circuits"
         (path "/1df96114-eb1a-4ddf-9ea3-acd2b4d12bf3/11663713-acec-45f1-8603-bba89fd94900"
-          (reference "R7") (unit 1)
-        )
-      )
+          (reference "R6") (unit 1)
+        )
+      )
