File: circuits/rbc_circuits.kicad_pcb (KiCad board)
At the start: 4 copper layers, 120 x 140 mm, 82 parts, among them IC1 BTN70301EPAXUMA1, IC2 BTN70301EPAXUMA1, IC3 BTN70301EPAXUMA1, IC4 BTN70301EPAXUMA1, IC5 BTN70301EPAXUMA1, IC6 BTN70301EPAXUMA1, IC7 BTN70301EPAXUMA1, IC8 BTN70301EPAXUMA1, J1 Conn_01x02_Pin, J2 Conn_01x02_Pin, J3 Conn_01x02_Pin, J4 Conn_01x06_Pin, J5 Conn_01x06_Pin, J6 Conn_01x02_Pin, J7 Conn_01x06_Pin, J8 Conn_01x06_Pin, J9 Conn_01x02_Pin, U1 TPS54202DDC

Commit message: PCB Rev2.0 publish
It's here
Parts:
- removed A1: A000067, A000067:ARDUINO_A000067
- removed the REF** at (163.8, 25.0)
- removed the REF** at (53.3, 25.0)
- removed the REF** at (53.3, 155.1)
- removed the REF** at (163.8, 155.1)
- added C15: 10nF, Capacitor_SMD:C_0805_2012Metric, F.Cu at (186.8, 109.4)
- added C16: 10nF, Capacitor_SMD:C_0805_2012Metric, F.Cu at (241.8, 158.8)
- added C17: 100uF, SamacSys_Parts:16SVF180M, F.Cu at (204.9, 107.6)
- added C18: 100uF, SamacSys_Parts:16SVF180M, F.Cu at (234.3, 175.4)
- added C19: 100nF, Capacitor_SMD:C_0402_1005Metric, F.Cu at (196.1, 140.7)
- added C20: 100nF, Capacitor_SMD:C_0402_1005Metric, F.Cu at (207.8, 143.8)
- added C21: 100nF, Capacitor_SMD:C_0402_1005Metric, F.Cu at (204.6, 160.2)
- added C22: 100nF, Capacitor_SMD:C_0402_1005Metric, F.Cu at (189.4, 146.5)
- added C23: 100nF, Capacitor_SMD:C_0402_1005Metric, F.Cu at (203.2, 161.5)
- added C24: 270uF, SamacSys_Parts:EEHZS1H221P, F.Cu at (157.7, 140.6)
- added C25: 100nF, Capacitor_SMD:C_0402_1005Metric, F.Cu at (155.4, 130.9)
- added C26: 10nF, Capacitor_SMD:C_0805_2012Metric, F.Cu at (142.3, 141.8)
- added C27: 100uF, SamacSys_Parts:16SVF180M, F.Cu at (149.8, 125.2)
- added C28: 220nF, Capacitor_SMD:C_0805_2012Metric, F.Cu at (182.3, 144.7)
- added C29: 220nF, Capacitor_SMD:C_0805_2012Metric, F.Cu at (183.9, 143.0)
- added C30: 100nF, Capacitor_SMD:C_0402_1005Metric, F.Cu at (201.0, 83.5)
- added C31: 100nF, Capacitor_SMD:C_0402_1005Metric, F.Cu at (139.9, 183.5)
- added C32: 220nF, Capacitor_SMD:C_0805_2012Metric, F.Cu at (185.6, 141.4)
- added C33: 100nF, Capacitor_SMD:C_0402_1005Metric, F.Cu at (257.1, 184.2)
- added D1: 450mV 3A, Diode_SMD:D_SMA, F.Cu at (165.5, 187.8)
- added D10: Red, Diode_SMD:D_0805_2012Metric, F.Cu at (187.2, 132.2)
- added D2: 450mV 3A, Diode_SMD:D_SMA, F.Cu at (184.5, 103.6)
- added D3: 450mV 3A, Diode_SMD:D_SMA, F.Cu at (247.9, 159.8)
- added D4: LED, Diode_SMD:D_0805_2012Metric, F.Cu at (200.1, 166.9)
- added D5: 450mV 3A, Diode_SMD:D_SMA, F.Cu at (136.1, 140.8)
- added D6: Green, Diode_SMD:D_0805_2012Metric, F.Cu at (212.7, 132.2)
- added D7: Green, Diode_SMD:D_0805_2012Metric, F.Cu at (206.3, 132.2)
- added D8: Green, Diode_SMD:D_0805_2012Metric, F.Cu at (200.0, 132.2)
- added D9: Green, Diode_SMD:D_0805_2012Metric, F.Cu at (193.5, 132.2)
- added G***: LOGO, LOGO, F.Cu at (183.9, 135.0)
- added G***: LOGO, LOGO, F.Cu at (196.8, 134.8)
- added G***: LOGO, LOGO, F.Cu at (190.5, 134.9)
- added G***: LOGO, LOGO, F.Cu at (203.2, 134.9)
- added G***: LOGO, LOGO, F.Cu at (209.6, 134.9)
- added G***: LOGO, decals:ugs, F.Cu at (229.9, 119.6)
- added G***: LOGO, LOGO, B.Cu at (200.0, 150.0)
- added IC10: BTN70301EPAXUMA1, rbc Custom Library:Infineon_PG-TSDSO-14-22_custom, F.Cu at (258.9, 176.8)
- added IC11: BTN70301EPAXUMA1, rbc Custom Library:Infineon_PG-TSDSO-14-22_custom, F.Cu at (252.1, 188.7)
- added IC9: BTN70301EPAXUMA1, rbc Custom Library:Infineon_PG-TSDSO-14-22_custom, F.Cu at (138.4, 176.9)
- added J10: Conn_01x06_Pin, Connector_Molex:Molex_Micro-Fit_3.0_43045-0612_2x03_P3.00mm_Vertical, F.Cu at (132.5, 191.4)
- added J11: Conn_01x06_Pin, Connector_Molex:Molex_Micro-Fit_3.0_43045-0612_2x03_P3.00mm_Vertical, F.Cu at (267.6, 186.6)
- added JP3: ON, Jumper:SolderJumper-2_P1.3mm_Open_RoundedPad1.0x1.5mm, F.Cu at (133.4, 148.1)
- added L2: 22uH, SamacSys_Parts:INDPM110100X400N, F.Cu at (160.1, 180.4)
- added L3: 22uH, SamacSys_Parts:INDPM110100X400N, F.Cu at (193.6, 102.6)
- added L4: 22uH, SamacSys_Parts:INDPM110100X400N, F.Cu at (244.3, 168.2)
- added L5: 10uH, Inductor_SMD:L_0805_2012Metric, F.Cu at (188.0, 148.3)
- added L6: 22uH, SamacSys_Parts:INDPM110100X400N, F.Cu at (139.8, 132.4)
- added R43: 4k7, Resistor_SMD:R_1206_3216Metric, F.Cu at (145.7, 174.3)
- added R44: 4k7, Resistor_SMD:R_1206_3216Metric, F.Cu at (220.3, 169.7)
- added R45: 4k7, Resistor_SMD:R_1206_3216Metric, F.Cu at (221.9, 173.9)
- added R46: 1k2, Resistor_SMD:R_1206_3216Metric, F.Cu at (224.6, 169.3)
- added R47: 4k7, Resistor_SMD:R_1206_3216Metric, F.Cu at (251.6, 174.3)
- added R48: 4k7, Resistor_SMD:R_1206_3216Metric, F.Cu at (253.1, 171.7)
- added R49: 4k7, Resistor_SMD:R_1206_3216Metric, F.Cu at (254.4, 169.5)
- added R50: 4k7, Resistor_SMD:R_1206_3216Metric, F.Cu at (243.4, 188.6)
- added R51: 4k7, Resistor_SMD:R_1206_3216Metric, F.Cu at (244.9, 185.9)
- added R52: 4k7, Resistor_SMD:R_1206_3216Metric, F.Cu at (246.2, 183.7)
- added REF**: MountingHole_4.3mm_M4, MountingHole:MountingHole_4.3mm_M4, F.Cu at (143.0, 206.0)
- added REF**: MountingHole_4.3mm_M4, MountingHole:MountingHole_4.3mm_M4, F.Cu at (143.0, 93.2)
- added REF**: MountingHole_4.3mm_M4, MountingHole:MountingHole_4.3mm_M4, F.Cu at (256.3, 93.2)
- added REF**: MountingHole_4.3mm_M4, MountingHole:MountingHole_4.3mm_M4, F.Cu at (256.3, 206.0)
- added S1: RESET, SamacSys_Parts:FSM4JSMATR, F.Cu at (210.3, 171.2)
- added U2: ATmega2560-16A, Package_QFP:TQFP-100_14x14mm_P0.5mm, F.Cu at (200.0, 150.0)
- C1: value 10uF -> 1uF; footprint Capacitor_SMD:C_1206_3216Metric_Pad1.33x1.80mm_HandSolder -> Capacitor_SMD:C_0603_1608Metric
- C10: value 100nF -> 100uF; footprint Capacitor_SMD:C_0603_1608Metric_Pad1.08x0.95mm_HandSolder -> SamacSys_Parts:16SVF180M
- C11, C12: value 220pF -> 270uF; footprint Capacitor_SMD:C_0402_1005Metric_Pad0.74x0.62mm_HandSolder -> SamacSys_Parts:EEHZS1H221P
- C13, C14: footprint Capacitor_SMD:C_0603_1608Metric_Pad1.08x0.95mm_HandSolder -> Capacitor_SMD:C_0402_1005Metric
- C2: value 0.1uF -> 270uF; footprint Capacitor_SMD:C_0603_1608Metric_Pad1.08x0.95mm_HandSolder -> SamacSys_Parts:EEHZS1H221P
- C3: value 0.1uF -> 4.7uF; footprint Capacitor_SMD:C_0603_1608Metric_Pad1.08x0.95mm_HandSolder -> Capacitor_SMD:C_1206_3216Metric
- C4: value 22uF -> 10nF; footprint Capacitor_SMD:C_1206_3216Metric_Pad1.33x1.80mm_HandSolder -> Capacitor_SMD:C_0402_1005Metric
- C5: value 22uF -> 100nF; footprint Capacitor_SMD:C_1206_3216Metric_Pad1.33x1.80mm_HandSolder -> Capacitor_SMD:C_0402_1005Metric
- C6: value 75pF -> 100nF; footprint Capacitor_SMD:C_0805_2012Metric_Pad1.18x1.45mm_HandSolder -> Capacitor_SMD:C_0402_1005Metric
- C7: value 220pF -> 10pF; footprint Capacitor_SMD:C_0402_1005Metric_Pad0.74x0.62mm_HandSolder -> Capacitor_SMD:C_0603_1608Metric
- C8: value 220pF -> 10nF; footprint Capacitor_SMD:C_0402_1005Metric_Pad0.74x0.62mm_HandSolder -> Capacitor_SMD:C_0805_2012Metric
- C9: value 100nF -> 22uF; footprint Capacitor_SMD:C_0603_1608Metric_Pad1.08x0.95mm_HandSolder -> Capacitor_SMD:C_1206_3216Metric
- IC1: value BTN70301EPAXUMA1 -> LT8609AEDDM#PBF; footprint rbc Custom Library:Infineon_PG-TSDSO-14-22_custom -> SamacSys_Parts:SON50P300X300X80-11N-D
- IC2, IC3, IC4, IC5: value BTN70301EPAXUMA1 -> LM2678SX-ADJ/NOPB; footprint rbc Custom Library:Infineon_PG-TSDSO-14-22_custom -> rbc Custom Library:KTW0007B_custom
- J2: value Conn_01x02_Pin -> Extra; footprint Connector_PinHeader_2.54mm:PinHeader_1x02_P2.54mm_Vertical -> Connector_PinHeader_2.54mm:PinHeader_2x02_P2.54mm_Vertical
- J3: value Conn_01x02_Pin -> ICSP; footprint Connector_PinHeader_2.54mm:PinHeader_1x02_P2.54mm_Vertical -> Connector_PinHeader_2.54mm:PinHeader_2x02_P2.54mm_Vertical
- J4: value Conn_01x06_Pin -> PROG; footprint Connector_Molex:Molex_Micro-Fit_3.0_43045-0612_2x03_P3.00mm_Vertical -> Connector_PinHeader_2.54mm:PinHeader_2x02_P2.54mm_Vertical
- J5: value Conn_01x06_Pin -> External Switch; footprint Connector_Molex:Molex_Micro-Fit_3.0_43045-0612_2x03_P3.00mm_Vertical -> TerminalBlock_Phoenix:TerminalBlock_Phoenix_MKDS-3-2-5.08_1x02_P5.08mm_Horizontal
- J6: value Conn_01x02_Pin -> Raspberry Pi Power/UART; footprint TerminalBlock_Phoenix:TerminalBlock_Phoenix_MKDS-3-2-5.08_1x02_P5.08mm_Horizontal -> Connector_Molex:Molex_Micro-Fit_3.0_43045-0612_2x03_P3.00mm_Vertical
- J7, J8: value Conn_01x06_Pin -> Extra 12V; footprint Connector_Molex:Molex_Micro-Fit_3.0_43045-0612_2x03_P3.00mm_Vertical -> Connector_Molex:Molex_Micro-Fit_3.0_43045-0412_2x02_P3.00mm_Vertical
- J9: value Conn_01x02_Pin -> Conn_01x06_Pin; footprint TerminalBlock_Phoenix:TerminalBlock_Phoenix_MKDS-3-2-5.08_1x02_P5.08mm_Horizontal -> Connector_Molex:Molex_Micro-Fit_3.0_43045-0612_2x03_P3.00mm_Vertical
- JP1: value SolderJumper_2_Open -> EN; footprint Jumper:SolderJumper-2_P1.3mm_Open_RoundedPad1.0x1.5mm -> Jumper:SolderJumper-3_P2.0mm_Open_TrianglePad1.0x1.5mm
- JP2: value D3087-98 -> SolderJumper_2_Open; footprint SamacSys_Parts:D308798 -> Jumper:SolderJumper-2_P1.3mm_Open_RoundedPad1.0x1.5mm
- L1: value 15uH -> 2.2uH; footprint LQH3NPH150MMEL:IND_LQH3NPH150MMEL -> SamacSys_Parts:INDC4441X200N
- R1: value 510k -> 18.2k; footprint Resistor_SMD:R_0805_2012Metric_Pad1.20x1.40mm_HandSolder -> Resistor_SMD:R_0603_1608Metric_Pad0.98x0.95mm_HandSolder
- R10, R20, R9: value 4k7 -> 8.87k; footprint Resistor_SMD:R_1206_3216Metric_Pad1.30x1.75mm_HandSolder -> Resistor_SMD:R_0603_1608Metric
- R11: value 1k2 -> 10k; footprint Resistor_SMD:R_1206_3216Metric_Pad1.30x1.75mm_HandSolder -> Resistor_SMD:R_0402_1005Metric
- R12: value 1k2 -> 1M; footprint Resistor_SMD:R_1206_3216Metric_Pad1.30x1.75mm_HandSolder -> Resistor_SMD:R_0402_1005Metric
- R13: value 4k7 -> 1k6; footprint Resistor_SMD:R_1206_3216Metric_Pad1.30x1.75mm_HandSolder -> Resistor_SMD:R_0805_2012Metric_Pad1.20x1.40mm_HandSolder
- R14: value 4k7 -> 3k3
- R15, R21, R22, R23, R24, R25: value 4k7 -> 300; footprint Resistor_SMD:R_1206_3216Metric_Pad1.30x1.75mm_HandSolder -> Resistor_SMD:R_0603_1608Metric_Pad0.98x0.95mm_HandSolder
- R16: value 4k7 -> 82k ±1%; footprint Resistor_SMD:R_1206_3216Metric_Pad1.30x1.75mm_HandSolder -> Resistor_SMD:R_0603_1608Metric_Pad0.98x0.95mm_HandSolder
- R17: value 4k7 -> 18k ±5%; footprint Resistor_SMD:R_1206_3216Metric_Pad1.30x1.75mm_HandSolder -> Resistor_SMD:R_0603_1608Metric_Pad0.98x0.95mm_HandSolder
- R18, R7, R8: value 4k7 -> 1k; footprint Resistor_SMD:R_1206_3216Metric_Pad1.30x1.75mm_HandSolder -> Resistor_SMD:R_0201_0603Metric
- R19: value 4k7 -> 10k; footprint Resistor_SMD:R_1206_3216Metric_Pad1.30x1.75mm_HandSolder -> Resistor_SMD:R_0402_1005Metric
- R2: value 49.9 -> 1k; footprint Resistor_SMD:R_0805_2012Metric_Pad1.20x1.40mm_HandSolder -> Resistor_SMD:R_0201_0603Metric
- R26, R27, R28, R30, R32, R33, R34, R35, R36, R37, R38, R39, R40, R41, R42: footprint Resistor_SMD:R_1206_3216Metric_Pad1.30x1.75mm_HandSolder -> Resistor_SMD:R_1206_3216Metric
- R29: value 1k2 -> 4k7; footprint Resistor_SMD:R_1206_3216Metric_Pad1.30x1.75mm_HandSolder -> Resistor_SMD:R_1206_3216Metric
- R3: value 100k -> 187k; footprint Resistor_SMD:R_1206_3216Metric_Pad1.30x1.75mm_HandSolder -> Resistor_SMD:R_0603_1608Metric
- R31: value 4k7 -> 1k2; footprint Resistor_SMD:R_1206_3216Metric_Pad1.30x1.75mm_HandSolder -> Resistor_SMD:R_1206_3216Metric
- R4: value 13.3k -> 8.87k; footprint Resistor_SMD:R_0805_2012Metric_Pad1.20x1.40mm_HandSolder -> Resistor_SMD:R_0603_1608Metric
- R5: value 1k6 -> 1M; footprint Resistor_SMD:R_0805_2012Metric_Pad1.20x1.40mm_HandSolder -> Resistor_SMD:R_0402_1005Metric
- R6: value 3k3 -> 100k; footprint Resistor_SMD:R_1206_3216Metric_Pad1.30x1.75mm_HandSolder -> Resistor_SMD:R_0201_0603Metric
- U1: value TPS54202DDC -> CSTCE16M0V53-R0; footprint Package_TO_SOT_SMD:SOT-23-6 -> SamacSys_Parts:CSTCE16M0V53R0
- moved J6 216.2 mm to (268.9, 127.5), turned to -60 degrees
- moved IC1 196.7 mm to (198.9, 210.8), turned to 0 degrees
- moved J5 195.5 mm to (249.4, 105.4), turned to 120 degrees
- moved R13 193.7 mm to (256.0, 138.8), turned to -60 degrees
- moved R14 193.6 mm to (258.1, 137.1), turned to 120 degrees
- moved C9 189.2 mm to (190.0, 201.8), turned to -90 degrees
- moved R10 183.5 mm to (248.9, 156.0), turned to 150 degrees
- moved C7 182.8 mm to (203.2, 214.8), turned to -90 degrees
- moved IC4 180.2 mm to (241.3, 148.1), turned to -30 degrees
- moved R8 179.7 mm to (244.6, 153.5), turned to -120 degrees
- moved R19 166.1 mm to (216.7, 143.0), turned to -60 degrees
- moved R11 155.6 mm to (204.5, 162.8), turned to -135 degrees
- moved R15 155.4 mm to (200.1, 164.8)
- moved R21 155.4 mm to (212.7, 135.7), turned to 90 degrees
- moved J4 155.1 mm to (180.8, 151.4)
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Connections:
- C1 pad 1: +BATT -> GND
- C1 pad 2: GND -> Net-(IC1-INTVCC)
- C10 pad 1: GND -> +12C
- C10 pad 2: +12V -> GND
- C11 pad 1: 4_IS -> +BATT
- C12 pad 1: 3_IS -> +BATT
- C13 pad 2: +12P -> +BATT
- C14 pad 2: +12P -> +BATT
- C3 pad 1: Net-(U1-BOOT) -> GND
- C3 pad 2: Net-(U1-SW) -> +BATT
- C4 pad 1: +5V -> GND
- C4 pad 2: GND -> Net-(IC1-TR/SS)
- C5 pad 1: +5V -> GND
- C5 pad 2: GND -> +BATT
- C6 pad 1: Net-(C6-Pad1) -> Net-(IC1-BST)
- C6 pad 2: Net-(U1-FB) -> Net-(IC1-SW)
- C7 pad 1: 1_IS -> Net-(IC1-FB)
- C7 pad 2: GND -> Net-(JP1-C)
- C8 pad 1: 2_IS -> Net-(D1-K)
- C8 pad 2: GND -> Net-(IC2-CB)
- C9 pad 1: +12V -> GND
- C9 pad 2: GND -> Net-(JP1-C)
- IC1 pad 1: unconnected-(IC1-NC_1-Pad1) -> Net-(IC1-BST)
- IC1 pad 10: 1_LOUT -> +BATT
- IC1 pad 11: unconnected-(IC1-NC_4-Pad11) -> GND
- IC1 pad 2: Net-(IC1-EN) -> Net-(IC1-SW)
- IC1 pad 3: Net-(IC1-DEN) -> Net-(IC1-INTVCC)
- IC1 pad 4: Net-(IC1-IS) -> Net-(IC1-RT)
- IC1 pad 5: unconnected-(IC1-NC_2-Pad5) -> Net-(IC1-INTVCC)
- IC1 pad 6: Net-(IC1-IN) -> Net-(IC1-FB)
- IC1 pad 7: unconnected-(IC1-NC_3-Pad7) -> Net-(IC1-TR/SS)
- IC1 pad 8: 1_LOUT -> Net-(IC1-PG)
- IC1 pad 9: 1_LOUT -> +BATT
- IC2 pad 1: unconnected-(IC2-NC_1-Pad1) -> Net-(D1-K)
- IC2 pad 2: Net-(IC2-EN) -> +BATT
- IC2 pad 3: Net-(IC2-DEN) -> Net-(IC2-CB)
- IC2 pad 4: Net-(IC2-IS) -> GND
- IC2 pad 6: Net-(IC2-IN) -> Net-(IC2-FB)
- IC2 pad 8: 2_LOUT -> unconnected-(IC2-TAB-Pad8)
- IC3 pad 1: unconnected-(IC3-NC_1-Pad1) -> Net-(D2-K)
- IC3 pad 2: Net-(IC3-EN) -> +BATT
- IC3 pad 3: Net-(IC3-DEN) -> Net-(IC3-CB)
- IC3 pad 4: Net-(IC1-IS) -> GND
- IC3 pad 6: Net-(IC3-IN) -> Net-(IC3-FB)
- IC3 pad 8: 1_ROUT -> unconnected-(IC3-TAB-Pad8)
- IC4 pad 1: unconnected-(IC4-NC_1-Pad1) -> Net-(D3-K)
- IC4 pad 2: Net-(IC4-EN) -> +BATT
- IC4 pad 3: Net-(IC4-DEN) -> Net-(IC4-CB)
- IC4 pad 4: Net-(IC2-IS) -> GND
- IC4 pad 6: Net-(IC4-IN) -> Net-(IC4-FB)
- IC4 pad 8: 2_ROUT -> unconnected-(IC4-TAB-Pad8)
- IC5 pad 1: unconnected-(IC5-NC_1-Pad1) -> Net-(D5-K)
- IC5 pad 2: Net-(IC5-EN) -> +BATT
- IC5 pad 3: Net-(IC5-DEN) -> Net-(IC5-CB)
- IC5 pad 4: Net-(IC5-IS) -> GND
- IC5 pad 6: Net-(IC5-IN) -> Net-(IC5-FB)
- IC5 pad 7: unconnected-(IC5-NC_3-Pad7) -> Net-(IC5-ON/~{OFF})
- IC5 pad 8: 4_LOUT -> unconnected-(IC5-TAB-Pad8)
- IC6 pad 10: 3_LOUT -> 1_LOUT
- IC6 pad 15: +12P -> +12V
- IC6 pad 8: 3_LOUT -> 1_LOUT
- IC6 pad 9: 3_LOUT -> 1_LOUT
- IC7 pad 10: 4_ROUT -> 2_LOUT
- IC7 pad 15: +12P -> +12C
- IC7 pad 4: Net-(IC5-IS) -> Net-(IC7-IS)
- IC7 pad 8: 4_ROUT -> 2_LOUT
- IC7 pad 9: 4_ROUT -> 2_LOUT
- IC8 pad 10: 3_ROUT -> 1_ROUT
- IC8 pad 15: +12P -> +12V
- IC8 pad 8: 3_ROUT -> 1_ROUT
- IC8 pad 9: 3_ROUT -> 1_ROUT
- J1 pad 1: Net-(J1-Pin_1) -> +BATT
- J2 pad 2: GND -> +5V
- J3 pad 1: PI_TX -> /MCU/MISO
- J3 pad 2: PI_RX -> /MCU/SCK
- J4 pad 1: 1_HALL_A -> /MCU/DTR
- J4 pad 2: +5V -> /MCU/PROG_RX
- J4 pad 3: 1_HALL_B -> /MCU/PROG_TX
- J4 pad 4: 1_LOUT -> EXTRA_A
- J5 pad 1: 2_HALL_A -> +5V
- J5 pad 2: +5V -> STOP
- J6 pad 1: +12V -> +5V
- J6 pad 2: GND -> +5V
- J7 pad 1: 4_HALL_A -> +12LF
- J7 pad 2: +5V -> +12LF
- J7 pad 3: 4_HALL_B -> GND
- J7 pad 4: 4_LOUT -> GND
- J8 pad 1: 3_HALL_A -> +12LF
- J8 pad 2: +5V -> +12LF
- J8 pad 3: 3_HALL_B -> GND
- J8 pad 4: 3_LOUT -> GND
- J9 pad 1: +12P -> 1_HALL_A
- J9 pad 2: GND -> +5V
- JP1 pad 1: Net-(JP1-A) -> +5V
- JP1 pad 2: Net-(JP1-B) -> Net-(JP1-C)
- JP2 pad 1: Net-(J1-Pin_1) -> BATT_LVL
- JP2 pad 2: +BATT -> Net-(JP2-B)
- L1 pad 1: Net-(U1-SW) -> Net-(IC1-SW)
- L1 pad 2: +5V -> Net-(JP1-C)
- R1 pad 1: +BATT -> Net-(IC1-RT)
- R1 pad 2: Net-(JP1-A) -> GND
- R10 pad 1: Net-(IC2-IS) -> +12P
- R10 pad 2: Net-(R10-Pad2) -> Net-(IC4-FB)
- R11 pad 1: GND -> +5V
- R11 pad 2: Net-(IC1-IS) -> /MCU/RESET
- R12 pad 1: GND -> Net-(U1-OUTPUT)
- R12 pad 2: Net-(IC2-IS) -> Net-(U1-INPUT)
- R13 pad 1: 1_LPWM -> Net-(U2-PJ1)
- R13 pad 2: Net-(IC1-IN) -> PI_RX
- R14 pad 1: +5V -> PI_RX
- R14 pad 2: Net-(IC1-DEN) -> GND
- R15 pad 1: +5V -> Net-(U2-PB7)
- R15 pad 2: Net-(IC1-EN) -> Net-(D4-A)
- R16 pad 1: 2_LPWM -> +BATT
- R16 pad 2: Net-(IC2-IN) -> Net-(JP2-B)
- R17 pad 1: +5V -> BATT_LVL
- R17 pad 2: Net-(IC2-DEN) -> GND
- R18 pad 1: +5V -> Net-(IC5-FB)
- R18 pad 2: Net-(IC2-EN) -> GND
- R19 pad 1: 1_RPWM -> STOP
- R19 pad 2: Net-(IC3-IN) -> GND
- R2 pad 1: +5V -> Net-(IC2-FB)
- R2 pad 2: Net-(C6-Pad1) -> GND
- R20 pad 1: Net-(IC3-DEN) -> +12LF
- R20 pad 2: +5V -> Net-(IC5-FB)
- R21 pad 1: Net-(IC3-EN) -> 5_BATT_IND
- R21 pad 2: +5V -> Net-(D6-A)
- R22 pad 1: 2_RPWM -> 4_BATT_IND
- R22 pad 2: Net-(IC4-IN) -> Net-(D7-A)
- R23 pad 1: Net-(IC4-DEN) -> 3_BATT_IND
- R23 pad 2: +5V -> Net-(D8-A)
- R24 pad 1: Net-(IC4-EN) -> 2_BATT_IND
- R24 pad 2: +5V -> Net-(D9-A)
- R25 pad 1: Net-(R25-Pad1) -> 1_BATT_IND
- R25 pad 2: 4_IS -> Net-(D10-A)
- R26 pad 2: 3_IS -> 1_IS
- R27 pad 1: Net-(IC5-IS) -> Net-(R27-Pad1)
- R27 pad 2: Net-(R25-Pad1) -> 2_IS
- R29 pad 1: GND -> Net-(IC7-IS)
- R29 pad 2: Net-(IC5-IS) -> Net-(R27-Pad1)
- R3 pad 1: Net-(C6-Pad1) -> Net-(IC1-FB)
- R3 pad 2: Net-(U1-FB) -> GND
- R31 pad 1: 4_LPWM -> GND
- R31 pad 2: Net-(IC5-IN) -> Net-(IC7-IS)
- R32 pad 1: +5V -> 1_LPWM
- R32 pad 2: Net-(IC5-DEN) -> Net-(IC6-IN)
- R33 pad 1: +5V -> M_EN_DEN
- R33 pad 2: Net-(IC5-EN) -> Net-(IC6-DEN)
- R34 pad 1: 3_LPWM -> M_EN_DEN
- R34 pad 2: Net-(IC6-IN) -> Net-(IC6-EN)
- R35 pad 1: +5V -> 2_LPWM
- R35 pad 2: Net-(IC6-DEN) -> Net-(IC7-IN)
- R36 pad 1: +5V -> M_EN_DEN
- R36 pad 2: Net-(IC6-EN) -> Net-(IC7-DEN)
- R37 pad 1: 4_RPWM -> M_EN_DEN
- R37 pad 2: Net-(IC7-IN) -> Net-(IC7-EN)
- R38 pad 1: Net-(IC7-DEN) -> 1_RPWM
- R38 pad 2: +5V -> Net-(IC8-IN)
- R39 pad 1: Net-(IC7-EN) -> Net-(IC8-DEN)
- R39 pad 2: +5V -> M_EN_DEN
- R4 pad 1: Net-(U1-FB) -> +12C
- R4 pad 2: GND -> Net-(IC2-FB)
- R40 pad 1: 3_RPWM -> Net-(IC8-EN)
- R40 pad 2: Net-(IC8-IN) -> M_EN_DEN
- R41 pad 1: Net-(IC8-DEN) -> 2_RPWM
- R41 pad 2: +5V -> Net-(IC9-IN)
- R42 pad 1: Net-(IC8-EN) -> Net-(IC9-DEN)
- R42 pad 2: +5V -> M_EN_DEN
- R5 pad 1: Net-(A1-Pad14) -> Net-(JP1-C)
- R5 pad 2: PI_RX -> Net-(IC1-FB)
- R6 pad 1: PI_RX -> Net-(JP1-C)
- R6 pad 2: GND -> Net-(IC1-PG)
- R7 pad 1: Net-(R7-Pad1) -> Net-(IC3-FB)
- R7 pad 2: 1_IS -> GND
- R8 pad 1: Net-(R10-Pad2) -> Net-(IC4-FB)
- R8 pad 2: 2_IS -> GND
- R9 pad 1: Net-(IC1-IS) -> +12V
- R9 pad 2: Net-(R7-Pad1) -> Net-(IC3-FB)
- U1 pad 1: GND -> Net-(U1-INPUT)
- U1 pad 2: Net-(U1-SW) -> GND
- U1 pad 3: +BATT -> Net-(U1-OUTPUT)
Routing:
- net M_EN_DEN: track 0.00 -> 296.7 mm, vias 0 -> 9
- net 4_HALL_B: track 96.7 -> 0.00 mm, vias 2 -> 0
- net 4_HALL_A: track 87.9 -> 0.00 mm, vias 2 -> 0
- net STOP: track 0.00 -> 73.7 mm, vias 0 -> 3
- net Net-(IC7-IS): track 0.00 -> 73.4 mm, vias 0 -> 2
- net Net-(IC10-IS): track 0.00 -> 73.4 mm, vias 0 -> 2
- net 4_IS: track 59.3 -> 0.00 mm, vias 1 -> 0
- net GND: track 3.97 -> 61.5 mm, vias 66 -> 231
- net Net-(U2-PJ1): track 0.00 -> 53.1 mm, vias 0 -> 2
- net Net-(A1-Pad14): track 50.2 -> 0.00 mm
- net 1_IS: track 0.00 -> 48.8 mm, vias 0 -> 2
- net /MCU/RESET: track 0.00 -> 46.8 mm, vias 0 -> 1
- net 3_LPWM: track 23.8 -> 69.2 mm, vias 0 -> 3
- net +12P: track 0.00 -> 44.2 mm, vias 16 -> 20
- net Net-(IC2-IS): track 40.6 -> 0.00 mm
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- added copper zone on B.Cu, net +12C
- added copper zone on F.Cu, net +12C
- added copper zone on F.Cu, net +12LF
- added copper zone on B.Cu, net +BATT
- added copper zone on B.Cu, net GND
- added copper zone on F.Cu, net Net-(D1-K)
- added copper zone on F.Cu, net Net-(D2-K)
- added copper zone on F.Cu, net Net-(D3-K)
- added copper zone on F.Cu, net Net-(D5-K)
- added copper zone on F.Cu, net Net-(IC1-INTVCC)
- added copper zone on F.Cu, net Net-(IC1-SW)
- added copper zone on F.Cu, net Net-(JP1-C)
- added copper zone on In2.Cu, net Net-(JP1-C)
- removed copper zone on F.Cu, net 1_IS
- removed copper zone on F.Cu, net 2_IS
- removed copper zone on F.Cu, net 4_LOUT
- removed copper zone on F.Cu, net 4_ROUT
- removed copper zone on F.Cu, net Net-(C6-Pad1)
- removed copper zone on F.Cu, net Net-(J1-Pin_1)
- removed copper zone on F.Cu, net Net-(U1-FB)
- removed copper zone on B.Cu, net Net-(U1-SW)
- removed copper zone on F.Cu, net Net-(U1-SW)
Other:
- board size 120 x 140 mm -> 171 x 171 mm
- board text added: "locked"
- board text added: "ロボットペニス!"
- board text removed: "MOTOR CONTROLLER PCB Rev 1.0"
- board text removed: "PROJECT RBC"
- board text removed: "© UGS 2023"
