File: circuits/utility.kicad_sch (KiCad schematic)
At the start: 0 parts

Commit message: PCB Rev2.0 publish
It's here
Parts:
- added C?: 100uF, SamacSys_Parts:16SVF180M, symbol Device:C_Polarized_Small
- added C?: 10nF, Capacitor_SMD:C_0805_2012Metric, symbol Device:C_Small
- added C?: 270uF, SamacSys_Parts:EEHZS1H221P, symbol Device:C_Polarized_Small
- added C?: 100nF, Capacitor_SMD:C_0402_1005Metric, symbol Device:C_Small
- added D?: 450mV 3A, Diode_SMD:D_SMA, symbol Device:D_Schottky_Small
- added D? (x4): Green, Diode_SMD:D_0805_2012Metric, symbol Device:LED
- added D?: Red, Diode_SMD:D_0805_2012Metric, symbol Device:LED
- added IC?: LM2678SX-ADJ/NOPB, rbc Custom Library:KTW0007B_custom, symbol SamacSys_Parts:LM2678SX-5.0_NOPB
- added J12: Raspberry Pi Power/UART, Connector_Molex:Molex_Micro-Fit_3.0_43045-0612_2x03_P3.00mm_Vertical, symbol Connector:Conn_01x06_Pin
- added J7, J8: Extra 12V, Connector_Molex:Molex_Micro-Fit_3.0_43045-0412_2x02_P3.00mm_Vertical, symbol Connector:Conn_01x04_Pin
- added J?: External Switch, TerminalBlock_Phoenix:TerminalBlock_Phoenix_MKDS-3-2-5.08_1x02_P5.08mm_Horizontal, symbol Connector:Conn_01x02_Pin
- added JP2: SolderJumper_2_Open, Jumper:SolderJumper-2_P1.3mm_Open_RoundedPad1.0x1.5mm, symbol Jumper:SolderJumper_2_Open
- added JP3: ON, Jumper:SolderJumper-2_P1.3mm_Open_RoundedPad1.0x1.5mm, symbol Jumper:SolderJumper_2_Open
- added L?: 22uH, SamacSys_Parts:INDPM110100X400N, symbol Device:L_Small
- added R16: 82k ±1%, Resistor_SMD:R_0603_1608Metric_Pad0.98x0.95mm_HandSolder, symbol Device:R_Small
- added R17: 18k ±5%, Resistor_SMD:R_0603_1608Metric_Pad0.98x0.95mm_HandSolder, symbol Device:R_Small
- added R19: 10k, Resistor_SMD:R_0402_1005Metric, symbol Device:R_Small
- added R? (x5): 300, Resistor_SMD:R_0603_1608Metric_Pad0.98x0.95mm_HandSolder, symbol Device:R_Small
- added R?: 8.87k, Resistor_SMD:R_0603_1608Metric, symbol Device:R_Small
- added R?: 1k, Resistor_SMD:R_0201_0603Metric, symbol Device:R_Small
Connections:
- new net: D?.2 (A), R?.2 (x5)
- new net: C?.1, D?.1 (K), IC?.1 (SWITCH_OUTPUT), L?.1
- new net: C?.2, IC?.3 (CB)
- new net: JP2.2 (B), R16.2
- new net: IC?.7 (ON/~{OFF}), JP3.2 (B)
- new net: IC?.6 (FB), R?.1, R?.2
- new net +12LF: C?.1, J7.1 (Pin_1), J7.2 (Pin_2), J8.1 (Pin_1), J8.2 (Pin_2), L?.2, R?.1
- new net +5V: J12.1 (Pin_1), J12.2 (Pin_2), J?.1 (Pin_1)
- new net +BATT: C?.1, C?.2, IC?.2 (INPUT), R16.1
- new net 1_BATT_IND: R?.1
- new net 2_BATT_IND: R?.1
- new net 3_BATT_IND: R?.1
- new net 4_BATT_IND: R?.1
- new net 5_BATT_IND: R?.1
- new net BATT_LVL: JP2.1 (A), R17.1
- new net GND: C?.1, C?.2, C?.2, D?.1 (K), D?.1 (K), D?.1 (K), D?.1 (K), D?.1 (K), D?.2 (A), IC?.4 (GND), J12.3 (Pin_3), J12.4 (Pin_4), J7.3 (Pin_3), J7.4 (Pin_4), J8.3 (Pin_3), J8.4 (Pin_4), JP3.1 (A), R17.2, R19.2, R?.2
- new net PI_RX: J12.5 (Pin_5)
- new net PI_TX: J12.6 (Pin_6)
- new net STOP: J?.2 (Pin_2), R19.1
- no-connect marks 0 -> 1
Other:
- note added: "12V regulator for LEDs"
- note added: "16SVPC100M"
- note added: "6S battery step-down"
- note added: "B340LA-13-F"
- note added: "CL21C103JBFNNNE"
- note added: "Emergency Stop Circuit"
- note added: "Short ON to switch off circuit"
- note added: "~4.536 max"
- title: (none) -> RBC by UGS
