Commit message: renaming

File: ros/rbc_navigation/description/robot_core.xacro (robot description, xacro)
@@ -12,5 +12,5 @@
         <origin xyz="0 0 0"/>
     </joint> launch-prefix="bash -c 'sleep 5; $0 $@'"
-    <!-- chassis description goes here. It describes the chassis of robocock which is a 54cm x 54cm x 150cm box -->
+    <!-- chassis description goes here. It describes the chassis of the bot which is a 54cm x 54cm x 150cm box -->
     <link name="chassis">
         <visual>
@@ -19,5 +19,5 @@
             <geometry>
                 <!-- <box size="0.54 0.54 1.5"/> -->
-                <mesh filename="package://robocock/meshes/frame_ultra_low_poly.stl"/>
+                <mesh filename="package://rbc_base/meshes/frame_ultra_low_poly.stl"/>
                 <!-- <mesh filename="model://frame_ultra_low_poly.stl"/> -->
             </geometry>

Commit message: update lidar position

File: ros/rbc_navigation/description/robot_core.xacro (robot description, xacro)
@@ -38,5 +38,5 @@
         <parent link="chassis"/>
         <child link="laser"/>
-        <origin xyz="-0.25 0 0.5" rpy="0 0 0"/>
+        <origin xyz="0 0 0.07" rpy="0 0 0"/>
     </joint>
     <link name="laser">

Commit message: fixed odometry

File: ros/rbc_navigation/description/robot_core.xacro (robot description, xacro)
@@ -38,5 +38,5 @@
         <parent link="chassis"/>
         <child link="laser"/>
-        <origin xyz="0 0 0.07" rpy="0 0 0"/>
+        <origin xyz="0 0 0.07" rpy="0 0 ${pi/2}"/>
     </joint>
     <link name="laser">
@@ -57,5 +57,5 @@
         <parent link="base_link"/>
         <child link="wheel_1"/>
-        <origin xyz="0.1575 0.1575 0" rpy="-${pi/2} 0 -${pi/4}"/>
+        <origin xyz="0.1575 -0.1575 0" rpy="-${pi/2} 0 ${pi/4}"/>
         <axis xyz="0 0 1"/>
     </joint>
@@ -89,5 +89,5 @@
         <parent link="base_link"/>
         <child link="wheel_2"/>
-        <origin xyz="0.1575 -0.1575 0" rpy="${pi/2} 0 ${pi/4}"/>
+        <origin xyz="0.1575 0.1575 0" rpy="${pi/2} 0 ${3*pi/4}"/>
         <axis xyz="0 0 -1"/>
     </joint>
@@ -121,5 +121,5 @@
         <parent link="base_link"/>
         <child link="wheel_3"/>
-        <origin xyz="-0.1575 0.1575 0" rpy="-${pi/2} 0 ${pi/4}"/>
+        <origin xyz="-0.1575 0.1575 0" rpy="-${pi/2} 0 ${5*pi/4}"/>
         <axis xyz="0 0 1"/>
     </joint>
@@ -153,5 +153,5 @@
         <parent link="base_link"/>
         <child link="wheel_4"/>
-        <origin xyz="-0.1575 -0.1575 0" rpy="${pi/2} 0 -${pi/4}"/>
+        <origin xyz="-0.1575 -0.1575 0" rpy="${pi/2} 0 ${7*pi/4}"/>
         <axis xyz="0 0 -1"/>
     </joint>

Commit message: updated wheel 1 coordinates

File: ros/rbc_navigation/description/robot_core.xacro (robot description, xacro)
@@ -53,9 +53,9 @@
         <material>Gazebo/White</material>
     </gazebo>
-    <!-- FRONT LEFT WHEEL AKA wheel_1 -->
+    <!-- WHEEL 1 (CLOCKWISE) -->
     <joint name="wheel_1_joint" type="continuous">
         <parent link="base_link"/>
         <child link="wheel_1"/>
-        <origin xyz="0.1575 -0.1575 0" rpy="-${pi/2} 0 ${pi/4}"/>
+        <origin xyz="0.2 0 0" rpy="-${pi/2} 0 ${pi/4}"/>
         <axis xyz="0 0 1"/>
     </joint>
@@ -85,5 +85,5 @@
         <maxContacts value= "1"/>
     </gazebo>
-    <!-- FRONT RIGHT WHEEL AKA wheel_2 -->
+    <!-- WHEEL 2 -->
     <joint name="wheel_2_joint" type="continuous">
         <parent link="base_link"/>
@@ -117,5 +117,5 @@
         <maxContacts value= "1"/>
     </gazebo>
-    <!-- REAR LEFT WHEEL AKA wheel_3 -->
+    <!-- WHEEL 3 -->
     <joint name="wheel_3_joint" type="continuous">
         <parent link="base_link"/>
@@ -141,36 +141,4 @@
     </link>
     <gazebo reference="wheel_3">
-        <material>Gazebo/Black</material>
-        <mu1 value="0.2"/>
-        <mu2 value="1.5"/>
-        <kp value="10000000.0" />
-        <kd value="10000.0" />
-        <fdir1 value="0 0 1"/>
-        <maxContacts value= "1"/>
-    </gazebo>
-    <!-- REAR RIGHT WHEEL AKA wheel_4 -->
-    <joint name="wheel_4_joint" type="continuous">
-        <parent link="base_link"/>
-        <child link="wheel_4"/>
-        <origin xyz="-0.1575 -0.1575 0" rpy="${pi/2} 0 ${7*pi/4}"/>
-        <axis xyz="0 0 -1"/>
-    </joint>
-    <link name="wheel_4">
-        <visual>
-            <geometry>
-                <cylinder length="0.038" radius="0.05" />
-            </geometry>
-            <material name="black"/>
-        </visual>
-        <collision>
-            <geometry>
-                <cylinder length="0.038" radius="0.05" />
-            </geometry>
-        </collision>
-        <xacro:inertial_cylinder mass="0.2" length="0.038" radius="0.05">
-            <origin xyz="0 0 0" rpy="0 0 0"/>
-        </xacro:inertial_cylinder>
-    </link>
-    <gazebo reference="wheel_4">
         <material>Gazebo/Black</material>
         <mu1 value="0.2"/>

Commit message: updated wheels xacro

File: ros/rbc_navigation/description/robot_core.xacro (robot description, xacro)
@@ -57,5 +57,5 @@
         <parent link="base_link"/>
         <child link="wheel_1"/>
-        <origin xyz="0.2 0 0" rpy="-${pi/2} 0 ${pi/4}"/>
+        <origin xyz="0.2 0 0" rpy="0 -${pi/2} 0"/>
         <axis xyz="0 0 1"/>
     </joint>
@@ -89,6 +89,6 @@
         <parent link="base_link"/>
         <child link="wheel_2"/>
-        <origin xyz="0.1575 0.1575 0" rpy="${pi/2} 0 ${3*pi/4}"/>
-        <axis xyz="0 0 -1"/>
+        <origin xyz="-0.1 -0.1732050808 0" rpy="0 ${pi/2} ${pi/3}"/>
+        <axis xyz="0 0 1"/>
     </joint>
     <link name="wheel_2">
@@ -121,5 +121,5 @@
         <parent link="base_link"/>
         <child link="wheel_3"/>
-        <origin xyz="-0.1575 0.1575 0" rpy="-${pi/2} 0 ${5*pi/4}"/>
+        <origin xyz="-0.1 0.1732050808 0" rpy="0 ${pi/2} -${pi/3}"/>
         <axis xyz="0 0 1"/>
     </joint>

Commit message: enabled slam

File: ros/rbc_navigation/description/robot_core.xacro (robot description, xacro)
@@ -19,5 +19,5 @@
             <geometry>
                 <!-- <box size="0.54 0.54 1.5"/> -->
-                <mesh filename="package://rbc_base/meshes/frame_ultra_low_poly.stl"/>
+                <mesh filename="package://rbc_base/meshes/frame_ultra_low_poly.dae"/>
                 <!-- <mesh filename="model://frame_ultra_low_poly.stl"/> -->
             </geometry>

Commit message: Update robot_core.xacro

File: ros/rbc_navigation/description/robot_core.xacro (robot description, xacro)
@@ -19,5 +19,5 @@
             <geometry>
                 <!-- <box size="0.54 0.54 1.5"/> -->
-                <mesh filename="package://rbc_base/meshes/frame_ultra_low_poly.dae"/>
+                <mesh filename="package://rbc_base/meshes/frame_ultra_low_poly.stl"/>
                 <!-- <mesh filename="model://frame_ultra_low_poly.stl"/> -->
             </geometry>

Commit message: mesh successfully loaded

File: ros/rbc_navigation/description/robot_core.xacro (robot description, xacro)
@@ -19,5 +19,5 @@
             <geometry>
                 <!-- <box size="0.54 0.54 1.5"/> -->
-                <mesh filename="package://rbc_base/meshes/frame_ultra_low_poly.stl"/>
+                <mesh filename="package://rbc_base/meshes/frame_ultra_low_poly.stl" scale="0.001 0.001 0.001"/>
                 <!-- <mesh filename="model://frame_ultra_low_poly.stl"/> -->
             </geometry>

Commit message: updated lidar location and orientation

File: ros/rbc_navigation/description/robot_core.xacro (robot description, xacro)
@@ -38,5 +38,5 @@
         <parent link="chassis"/>
         <child link="laser"/>
-        <origin xyz="0 0 0.07" rpy="0 0 ${pi/2}"/>
+        <origin xyz="0 0 0.07" rpy="0 0 0"/>
     </joint>
     <link name="laser">

Commit message: updated chassis inertial and collision model

File: ros/rbc_navigation/description/robot_core.xacro (robot description, xacro)
@@ -26,12 +26,13 @@
         <!-- physics model -->
         <collision>
-            <origin xyz="0 0 0.75" rpy="0 0 0"/>
+            <origin xyz="0 0 0.77" rpy="0 0 0"/>
             <geometry>
-                <box size="0.54 0.54 1.5"/>
+                <cylinder length="1.54" radius="0.25"/>
             </geometry>
         </collision>
-        <xacro:inertial_box mass="10" x="0.54" y="0.54" z="1.5">
-            <origin xyz="0 0 0.75" rpy="0 0 0"/>
-        </xacro:inertial_box>
+        <!-- <xacro:inertial_box mass="10" x="0.54" y="0.54" z="1.5"> -->
+        <xacro:inertial_cylinder mass="20" length="1.54" radius="0.25">
+            <origin xyz="0 0 0.77" rpy="0 0 0"/>
+        </xacro:inertial_cylinder>
     </link>
     <joint name="laser_joint" type="fixed">

Commit message: changed messages to 3 wheels

File: ros/rbc_navigation/description/robot_core.xacro (robot description, xacro)
@@ -180,14 +180,4 @@
         </actuator>
     </transmission>
-    <transmission name="tran4">
-        <type>transmission_interface/SimpleTransmission</type>
-        <joint name="wheel_4_joint">
-            <hardwareInterface>hardware_interface/VelocityJointInterface</hardwareInterface>
-        </joint>
-        <actuator name="motor_4">
-            <hardwareInterface>VelocityJointInterface</hardwareInterface>
-            <mechanicalReduction>1</mechanicalReduction>
-        </actuator>
-    </transmission>
     <gazebo>
         <plugin name="gazebo_ros_control" filename="libgazebo_ros_control.so">
